File: Circuit/Mala.kicad_pcb (KiCad board)
At the start: 2 copper layers, 89 parts, among them J1 CONN_01X01, J10 CONN_01X01, J11 CONN_01X01, J12 CONN_01X01, J13 CONN_01X01, J14 CONN_01X01, J15 CONN_01X01, J16 CONN_01X01, J17 CONN_01X01, J18 CONN_01X01, J19 CONN_01X01, J2 CONN_01X01, J20 CONN_01X01, J21 CONN_01X01, J22 CONN_01X01, J23 CONN_01X01, J24 CONN_01X01, J25 CONN_01X01, J26 CONN_01X01, J27 CONN_01X01, J28 CONN_01X01, J29 CONN_01X01, J3 CONN_01X01, J30 CONN_01X01, J31 CONN_01X01, J32 CONN_01X01, J33 CONN_01X01, J4 CONN_01X01, J5 CONN_01X01, J6 CONN_02X08, J7 CONN_01X01, J8 CONN_01X01, J9 CONN_01X01, Q1 Q_NMOS_GSD, Q10 Q_NMOS_GSD, Q11 Q_NMOS_GSD, Q12 Q_NMOS_GSD, Q13 Q_NMOS_GSD, Q14 Q_NMOS_GSD, Q15 Q_NMOS_GSD, Q16 Q_NMOS_GSD, Q17 Q_NMOS_GSD, Q18 Q_NMOS_GSD, Q19 Q_NMOS_GSD, Q2 Q_NMOS_GSD, Q20 Q_NMOS_GSD, Q21 Q_NMOS_GSD, Q22 Q_NMOS_GSD, Q23 Q_NMOS_GSD, Q24 Q_NMOS_GSD, Q25 Q_NMOS_GSD, Q26 Q_NMOS_GSD, Q27 Q_NMOS_GSD, Q28 Q_NMOS_GSD, Q29 Q_NMOS_GSD, Q3 Q_NMOS_GSD, Q30 Q_NMOS_GSD, Q31 Q_NMOS_GSD, Q32 Q_NMOS_GSD, Q33 Q_NMOS_GSD, Q34 Q_NMOS_GSD, Q35 Q_NMOS_GSD, Q36 Q_NMOS_GSD, Q37 Q_NMOS_GSD, Q38 Q_NMOS_GSD, Q39 Q_NMOS_GSD, Q4 Q_NMOS_GSD, Q40 Q_NMOS_GSD, Q5 Q_NMOS_GSD, Q6 Q_NMOS_GSD, Q7 Q_NMOS_GSD, Q8 Q_NMOS_GSD, Q9 Q_NMOS_GSD

Commit message: c
Parts:
- moved C8 94.0 mm to (141.0, 125.7)
- moved C6 67.3 mm to (104.1, 141.0)
- moved R6 63.1 mm to (102.9, 148.6)
- moved Q26 40.4 mm to (106.9, 144.2)
- moved Q35 36.9 mm to (86.4, 142.2)
- moved Q36 36.9 mm to (95.2, 142.2)
- moved Q25 36.9 mm to (97.5, 136.0)
- moved Q24 36.0 mm to (88.1, 135.1)
- moved Q39 35.9 mm to (116.8, 121.9)
- moved Q32 33.0 mm to (116.8, 114.3)
- moved Q40 29.4 mm to (124.5, 121.9)
- moved R5 25.4 mm to (127.5, 92.9)
- moved C5 25.4 mm to (129.4, 85.7)
- moved Q33 24.6 mm to (125.7, 114.3)
- moved Q34 23.6 mm to (132.1, 121.9)
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Changed lines of the file:
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@@
   (general
     (links 149)
-    (no_connects 124)
+    (no_connects 135)
     (area 34.336667 34.795 253.953334 171.485)
     (thickness 1.6)
@@
   )
   (module Capacitors_SMD:C_0603_HandSoldering (layer F.Cu)
-    (at 154.813 86.995)
+    (at 129.413 85.725)
     (descr "Capacitor SMD 0603, hand soldering")
     (tags "capacitor 0603")
@@
   )
   (module Capacitors_SMD:C_0603_HandSoldering (layer F.Cu)
-    (at 165.354 112.903)
+    (at 104.14 140.97)
     (descr "Capacitor SMD 0603, hand soldering")
     (tags "capacitor 0603")
@@
   )
   (module Capacitors_SMD:C_0603_HandSoldering (layer F.Cu)
-    (at 52.07 156.21)
+    (at 140.97 125.73)
     (descr "Capacitor SMD 0603, hand soldering")
     (tags "capacitor 0603")
@@
   )
   (module TO_SOT_Packages_SMD:SOT-23_Handsoldering (layer F.Cu)
-    (at 122.7582 83.312 180)
+    (at 110.0582 82.042 180)
     (descr "SOT-23, Handsoldering")
     (tags SOT-23)
@@
   )
   (module TO_SOT_Packages_SMD:SOT-23_Handsoldering (layer F.Cu)
-    (at 130.1115 83.2866)
+    (at 117.4115 82.0166)
     (descr "SOT-23, Handsoldering")
     (tags SOT-23)
@@
   )
   (module TO_SOT_Packages_SMD:SOT-23_Handsoldering (layer F.Cu)
-    (at 140.5636 81.5213)
+    (at 127.8636 80.2513)
     (descr "SOT-23, Handsoldering")
     (tags SOT-23)
@@
   )
   (module TO_SOT_Packages_SMD:SOT-23_Handsoldering (layer F.Cu)
-    (at 114.7318 110.9853 180)
+    (at 88.0618 135.1153 180)
     (descr "SOT-23, Handsoldering")
     (tags SOT-23)
@@
   )
   (module TO_SOT_Packages_SMD:SOT-23_Handsoldering (layer F.Cu)
-    (at 125.3998 111.8743)
+    (at 97.4598 136.0043)
     (descr "SOT-23, Handsoldering")
     (tags SOT-23)
@@
   )
   (module TO_SOT_Packages_SMD:SOT-23_Handsoldering (layer F.Cu)
-    (at 134.8613 114.9858)
+    (at 106.9213 144.1958)
     (descr "SOT-23, Handsoldering")
     (tags SOT-23)
@@
   )
   (module TO_SOT_Packages_SMD:SOT-23_Handsoldering (layer F.Cu)
-    (at 148.5011 105.0036)
+    (at 142.24 104.14)
     (descr "SOT-23, Handsoldering")
     (tags SOT-23)
@@
   )
   (module TO_SOT_Packages_SMD:SOT-23_Handsoldering (layer F.Cu)
-    (at 122.8725 88.519 180)
+    (at 110.1725 87.249 180)
     (descr "SOT-23, Handsoldering")
     (tags SOT-23)
@@
   )
   (module TO_SOT_Packages_SMD:SOT-23_Handsoldering (layer F.Cu)
-    (at 130.5306 88.8619)
+    (at 117.8306 87.5919)
     (descr "SOT-23, Handsoldering")
     (tags SOT-23)
@@
   )
   (module TO_SOT_Packages_SMD:SOT-23_Handsoldering (layer F.Cu)
-    (at 148.5011 105.0036)
+    (at 149.86 116.84)
     (descr "SOT-23, Handsoldering")
     (tags SOT-23)
@@
   )
   (module TO_SOT_Packages_SMD:SOT-23_Handsoldering (layer F.Cu)
-    (at 148.5011 105.0036)
+    (at 116.84 114.3)
     (descr "SOT-23, Handsoldering")
     (tags SOT-23)
@@
   )
   (module TO_SOT_Packages_SMD:SOT-23_Handsoldering (layer F.Cu)
-    (at 148.5011 105.0036)
+    (at 125.73 114.3)
     (descr "SOT-23, Handsoldering")
     (tags SOT-23)
@@
   )
   (module TO_SOT_Packages_SMD:SOT-23_Handsoldering (layer F.Cu)
-    (at 148.5011 105.0036)
+    (at 132.08 121.92)
     (descr "SOT-23, Handsoldering")
     (tags SOT-23)
@@
   )
   (module TO_SOT_Packages_SMD:SOT-23_Handsoldering (layer F.Cu)
-    (at 114.3 118.11 180)
+    (at 86.36 142.24 180)
     (descr "SOT-23, Handsoldering")
     (tags SOT-23)
@@
   )
   (module TO_SOT_Packages_SMD:SOT-23_Handsoldering (layer F.Cu)
-    (at 123.19 118.11)
+    (at 95.25 142.24)
     (descr "SOT-23, Handsoldering")
     (tags SOT-23)
@@
   )
   (module TO_SOT_Packages_SMD:SOT-23_Handsoldering (layer F.Cu)
-    (at 148.5011 105.0036)
+    (at 153.67 101.6)
     (descr "SOT-23, Handsoldering")
     (tags SOT-23)
@@
   )
   (module TO_SOT_Packages_SMD:SOT-23_Handsoldering (layer F.Cu)
-    (at 148.5011 105.0036)
+    (at 153.67 110.49)
     (descr "SOT-23, Handsoldering")
     (tags SOT-23)
@@
   )
   (module TO_SOT_Packages_SMD:SOT-23_Handsoldering (layer F.Cu)
-    (at 148.5011 105.0036)
+    (at 116.84 121.92)
     (descr "SOT-23, Handsoldering")
     (tags SOT-23)
@@
   )
   (module TO_SOT_Packages_SMD:SOT-23_Handsoldering (layer F.Cu)
-    (at 148.5011 105.0036)
+    (at 124.46 121.92)
     (descr "SOT-23, Handsoldering")
     (tags SOT-23)
@@
   )
   (module Resistors_SMD:R_0603_HandSoldering (layer F.Cu)
-    (at 152.8826 94.2086)
+    (at 127.4826 92.9386)
     (descr "Resistor SMD 0603, hand soldering")
     (tags "resistor 0603")
@@
   )
   (module Resistors_SMD:R_0603_HandSoldering (layer F.Cu)
-    (at 148.5011 105.0036)
+    (at 102.87 148.59)
     (descr "Resistor SMD 0603, hand soldering")
     (tags "resistor 0603")
@@
   )
   (module Resistors_SMD:R_0603_HandSoldering (layer F.Cu)
-    (at 148.5011 105.0036)
+    (at 142.24 111.76)
     (descr "Resistor SMD 0603, hand soldering")
     (tags "resistor 0603")
@@
   )
   (module Resistors_SMD:R_0603_HandSoldering (layer F.Cu)
-    (at 148.5011 105.0036)
+    (at 133.35 114.3)
     (descr "Resistor SMD 0603, hand soldering")
     (tags "resistor 0603")

Commit message: c
Parts:
- moved J22 132.0 mm to (82.5, 167.6)
- moved J24 132.0 mm to (82.5, 167.6)
- moved J25 132.0 mm to (82.5, 167.6)
- moved J26 132.0 mm to (82.5, 167.6)
- moved J27 132.0 mm to (82.5, 167.6)
- moved J28 132.0 mm to (82.5, 167.6)
- moved J29 132.0 mm to (82.5, 167.6)
- moved J30 132.0 mm to (82.5, 167.6)
- moved J31 132.0 mm to (82.5, 167.6)
- moved J32 132.0 mm to (82.5, 167.6)
- moved J33 132.0 mm to (82.5, 167.6)
- moved J23 85.4 mm to (100.3, 111.8)
- moved R8 14.4 mm to (123.2, 124.5)
- moved Q39 9.92 mm to (110.5, 114.3), turned to 180 degrees
- moved Q32 9.92 mm to (109.2, 108.0), turned to 180 degrees
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Changed lines of the file:
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@@
   (general
     (links 149)
-    (no_connects 135)
+    (no_connects 136)
     (area 34.336667 34.795 253.953334 171.485)
     (thickness 1.6)
@@
   )
   (module TO_SOT_Packages_SMD:SOT-23_Handsoldering (layer F.Cu)
-    (at 116.84 114.3)
+    (at 109.22 107.95 180)
     (descr "SOT-23, Handsoldering")
     (tags SOT-23)
     (attr smd)
-    (fp_text reference Q32 (at 0 -2.5) (layer F.SilkS)
+    (fp_text reference Q32 (at 0 -2.5 180) (layer F.SilkS)
       (effects (font (size 1 1) (thickness 0.15)))
     )
-    (fp_text value Q_NMOS_GSD (at 0 2.5) (layer F.Fab)
+    (fp_text value Q_NMOS_GSD (at 0 2.5 180) (layer F.Fab)
       (effects (font (size 1 1) (thickness 0.15)))
     )
-    (fp_text user %R (at 0 0 90) (layer F.Fab)
+    (fp_text user %R (at 0 0 270) (layer F.Fab)
       (effects (font (size 0.5 0.5) (thickness 0.075)))
     )
@@
     (fp_line (start -0.7 1.52) (end 0.7 1.52) (layer F.Fab) (width 0.1))
     (fp_line (start 0.76 1.58) (end -0.7 1.58) (layer F.SilkS) (width 0.12))
-    (pad 1 smd rect (at -1.5 -0.95) (size 1.9 0.8) (layers F.Cu F.Paste F.Mask)
+    (pad 1 smd rect (at -1.5 -0.95 180) (size 1.9 0.8) (layers F.Cu F.Paste F.Mask)
       (net 19 С4))
-    (pad 2 smd rect (at -1.5 0.95) (size 1.9 0.8) (layers F.Cu F.Paste F.Mask)
+    (pad 2 smd rect (at -1.5 0.95 180) (size 1.9 0.8) (layers F.Cu F.Paste F.Mask)
       (net 47 "Net-(Q32-Pad2)"))
-    (pad 3 smd rect (at 1.5 0) (size 1.9 0.8) (layers F.Cu F.Paste F.Mask)
+    (pad 3 smd rect (at 1.5 0 180) (size 1.9 0.8) (layers F.Cu F.Paste F.Mask)
       (net 23 Vcntrl))
     (model ${KISYS3DMOD}/TO_SOT_Packages_SMD.3dshapes\SOT-23.wrl
@@
   )
   (module TO_SOT_Packages_SMD:SOT-23_Handsoldering (layer F.Cu)
-    (at 125.73 114.3)
+    (at 118.11 107.95)
     (descr "SOT-23, Handsoldering")
     (tags SOT-23)
@@
   )
   (module TO_SOT_Packages_SMD:SOT-23_Handsoldering (layer F.Cu)
-    (at 132.08 121.92)
+    (at 128.27 113.03)
     (descr "SOT-23, Handsoldering")
     (tags SOT-23)
@@
   )
   (module TO_SOT_Packages_SMD:SOT-23_Handsoldering (layer F.Cu)
-    (at 116.84 121.92)
+    (at 110.49 114.3 180)
     (descr "SOT-23, Handsoldering")
     (tags SOT-23)
     (attr smd)
-    (fp_text reference Q39 (at 0 -2.5) (layer F.SilkS)
+    (fp_text reference Q39 (at 0 -2.5 180) (layer F.SilkS)
       (effects (font (size 1 1) (thickness 0.15)))
     )
-    (fp_text value Q_NMOS_GSD (at 0 2.5) (layer F.Fab)
+    (fp_text value Q_NMOS_GSD (at 0 2.5 180) (layer F.Fab)
       (effects (font (size 1 1) (thickness 0.15)))
     )
-    (fp_text user %R (at 0 0 90) (layer F.Fab)
+    (fp_text user %R (at 0 0 270) (layer F.Fab)
       (effects (font (size 0.5 0.5) (thickness 0.075)))
     )
@@
     (fp_line (start -0.7 1.52) (end 0.7 1.52) (layer F.Fab) (width 0.1))
     (fp_line (start 0.76 1.58) (end -0.7 1.58) (layer F.SilkS) (width 0.12))
-    (pad 1 smd rect (at -1.5 -0.95) (size 1.9 0.8) (layers F.Cu F.Paste F.Mask)
+    (pad 1 smd rect (at -1.5 -0.95 180) (size 1.9 0.8) (layers F.Cu F.Paste F.Mask)
       (net 19 С4))
-    (pad 2 smd rect (at -1.5 0.95) (size 1.9 0.8) (layers F.Cu F.Paste F.Mask)
+    (pad 2 smd rect (at -1.5 0.95 180) (size 1.9 0.8) (layers F.Cu F.Paste F.Mask)
       (net 51 "Net-(Q39-Pad2)"))
-    (pad 3 smd rect (at 1.5 0) (size 1.9 0.8) (layers F.Cu F.Paste F.Mask)
+    (pad 3 smd rect (at 1.5 0 180) (size 1.9 0.8) (layers F.Cu F.Paste F.Mask)
       (net 24 Vfb))
     (model ${KISYS3DMOD}/TO_SOT_Packages_SMD.3dshapes\SOT-23.wrl
@@
   )
   (module TO_SOT_Packages_SMD:SOT-23_Handsoldering (layer F.Cu)
-    (at 124.46 121.92)
+    (at 118.11 114.3)
     (descr "SOT-23, Handsoldering")
     (tags SOT-23)
@@
   )
   (module Resistors_SMD:R_0603_HandSoldering (layer F.Cu)
-    (at 133.35 114.3)
+    (at 123.19 124.46)
     (descr "Resistor SMD 0603, hand soldering")
     (tags "resistor 0603")
@@
   )
   (module Pin_Headers:Pin_Header_Straight_1x01_Pitch2.54mm (layer F.Cu)
-    (at 57.15 38.1)
+    (at 82.55 167.64)
     (descr "Through hole straight pin header, 1x01, 2.54mm pitch, single row")
     (tags "Through hole pin header THT 1x01 2.54mm single row")
@@
   )
   (module Pin_Headers:Pin_Header_Straight_1x01_Pitch2.54mm (layer F.Cu)
-    (at 57.15 38.1)
+    (at 100.33 111.76)
     (descr "Through hole straight pin header, 1x01, 2.54mm pitch, single row")
     (tags "Through hole pin header THT 1x01 2.54mm single row")
@@
   )
   (module Pin_Headers:Pin_Header_Straight_1x01_Pitch2.54mm (layer F.Cu)
-    (at 57.15 38.1)
+    (at 82.55 167.64)
     (descr "Through hole straight pin header, 1x01, 2.54mm pitch, single row")
     (tags "Through hole pin header THT 1x01 2.54mm single row")
@@
   )
   (module Pin_Headers:Pin_Header_Straight_1x01_Pitch2.54mm (layer F.Cu)
-    (at 57.15 38.1)
+    (at 82.55 167.64)
     (descr "Through hole straight pin header, 1x01, 2.54mm pitch, single row")
     (tags "Through hole pin header THT 1x01 2.54mm single row")
@@
   )
   (module Pin_Headers:Pin_Header_Straight_1x01_Pitch2.54mm (layer F.Cu)
-    (at 57.15 38.1)
+    (at 82.55 167.64)
     (descr "Through hole straight pin header, 1x01, 2.54mm pitch, single row")
     (tags "Through hole pin header THT 1x01 2.54mm single row")
@@
   )
   (module Pin_Headers:Pin_Header_Straight_1x01_Pitch2.54mm (layer F.Cu)
-    (at 57.15 38.1)
+    (at 82.55 167.64)
     (descr "Through hole straight pin header, 1x01, 2.54mm pitch, single row")
     (tags "Through hole pin header THT 1x01 2.54mm single row")
@@
   )
   (module Pin_Headers:Pin_Header_Straight_1x01_Pitch2.54mm (layer F.Cu)
-    (at 57.15 38.1)
+    (at 82.55 167.64)
     (descr "Through hole straight pin header, 1x01, 2.54mm pitch, single row")
     (tags "Through hole pin header THT 1x01 2.54mm single row")
@@
   )
   (module Pin_Headers:Pin_Header_Straight_1x01_Pitch2.54mm (layer F.Cu)
-    (at 57.15 38.1)
+    (at 82.55 167.64)
     (descr "Through hole straight pin header, 1x01, 2.54mm pitch, single row")
     (tags "Through hole pin header THT 1x01 2.54mm single row")
@@
   )
   (module Pin_Headers:Pin_Header_Straight_1x01_Pitch2.54mm (layer F.Cu)
-    (at 57.15 38.1)
+    (at 82.55 167.64)
     (descr "Through hole straight pin header, 1x01, 2.54mm pitch, single row")
     (tags "Through hole pin header THT 1x01 2.54mm single row")
@@
   )
   (module Pin_Headers:Pin_Header_Straight_1x01_Pitch2.54mm (layer F.Cu)
-    (at 57.15 38.1)
+    (at 82.55 167.64)
     (descr "Through hole straight pin header, 1x01, 2.54mm pitch, single row")
     (tags "Through hole pin header THT 1x01 2.54mm single row")
@@
   )
   (module Pin_Headers:Pin_Header_Straight_1x01_Pitch2.54mm (layer F.Cu)
-    (at 57.15 38.1)
+    (at 82.55 167.64)
     (descr "Through hole straight pin header, 1x01, 2.54mm pitch, single row")
     (tags "Through hole pin header THT 1x01 2.54mm single row")
@@
   )
   (module Pin_Headers:Pin_Header_Straight_1x01_Pitch2.54mm (layer F.Cu)
-    (at 57.15 38.1)
+    (at 82.55 167.64)
     (descr "Through hole straight pin header, 1x01, 2.54mm pitch, single row")
     (tags "Through hole pin header THT 1x01 2.54mm single row")

Commit message: c
Parts:
- moved J9 106.5 mm to (106.7, 123.2)
- moved J5 97.0 mm to (152.4, 114.3)
- moved J12 75.0 mm to (114.3, 111.8)
- moved J22 68.2 mm to (115.6, 108.0)
- moved J31 66.5 mm to (111.8, 108.0)
- moved Q24 39.7 mm to (118.7, 109.9), turned to 90 degrees
- moved Q35 39.3 mm to (108.6, 109.9), turned to 90 degrees
- moved R6 34.5 mm to (113.0, 115.6)
- moved J30 33.5 mm to (96.5, 137.2)
- moved Q36 29.3 mm to (108.6, 116.2), turned to 270 degrees
- moved Q25 29.1 mm to (118.7, 116.2), turned to 270 degrees
- moved C6 25.6 mm to (115.6, 118.1), turned to 180 degrees
- moved R8 23.4 mm to (146.1, 119.4)
- moved Q26 23.1 mm to (113.0, 121.9), turned to 270 degrees
- moved Q39 21.9 mm to (132.1, 118.1)
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
Commit message: c
Parts:
- moved J32 110.8 mm to (132.1, 68.6)
- moved J33 106.6 mm to (121.9, 68.6)
- moved J24 103.2 mm to (106.7, 67.3)
- moved J25 103.2 mm to (106.7, 67.3)
- moved J26 103.2 mm to (106.7, 67.3)
- moved J27 103.2 mm to (106.7, 67.3)
- moved J28 103.2 mm to (106.7, 67.3)
- moved J29 103.2 mm to (106.7, 67.3)
- moved J8 93.9 mm to (167.6, 59.7)
- moved J13 89.8 mm to (128.3, 86.4)
- moved C7 85.6 mm to (132.1, 83.8), turned to 270 degrees
- moved J7 65.9 mm to (143.5, 86.4)
- moved Q38 55.4 mm to (120.7, 88.9)
- moved Q37 48.5 mm to (114.3, 88.9), turned to 180 degrees
- moved R5 44.5 mm to (163.8, 67.3), turned to 90 degrees
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
Commit message: c
Parts:
- moved J10 77.1 mm to (122.2, 116.3)
- moved J24 54.6 mm to (100.8, 121.6)
- moved J29 52.9 mm to (110.1, 120.1)
- moved C5 36.2 mm to (135.3, 85.7)
- moved R5 36.2 mm to (135.3, 89.5)
- moved J22 34.8 mm to (150.4, 106.8)
- moved Q30 34.4 mm to (130.8, 92.1)
- moved Q29 33.8 mm to (124.5, 92.1)
- moved J32 33.8 mm to (109.9, 94.0)
- moved J8 33.8 mm to (145.4, 85.1)
- moved Q23 33.8 mm to (146.7, 91.4)
- moved Q35 32.6 mm to (141.2, 109.2)
- moved R6 32.4 mm to (145.4, 115.5)
- moved Q22 32.2 mm to (130.8, 83.8)
- moved Q36 32.2 mm to (140.8, 115.9)
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Routing:
- net Vfb: track 0.00 -> 11.4 mm
- net Vcntrl: track 0.00 -> 10.8 mm
- net GND: track 0.00 -> 5.81 mm
- net Net-(Q34-Pad2): track 0.00 -> 5.80 mm
- net Net-(C8-Pad1): track 0.00 -> 5.80 mm
- net Net-(Q17-Pad2): track 0.00 -> 5.76 mm
- net Net-(Q7-Pad2): track 0.00 -> 4.17 mm
- net Net-(Q32-Pad2): track 0.00 -> 4.14 mm
- net Net-(Q39-Pad2): track 0.00 -> 4.14 mm
- net (no net): track 0.00 -> 0.75 mm
- added copper zone on F.Cu, net С0
- added copper zone on F.Cu, net С2
- added copper zone on F.Cu, net С4

Commit message: c
Parts:
- moved J12 9.08 mm to (148.1, 121.3)
- moved J31 4.29 mm to (141.2, 104.5)
- moved J22 2.23 mm to (149.5, 104.8)
- moved Q24 1.65 mm to (149.3, 109.8)
- moved Q25 1.65 mm to (150.1, 116.3)
Routing:
- net GND: track 5.81 -> 17.7 mm
- net Net-(Q35-Pad2): track 0.00 -> 4.60 mm
- net Net-(Q24-Pad2): track 0.00 -> 3.92 mm
- net Vcntrl: track 10.8 -> 14.4 mm
- net Vfb: track 11.4 -> 14.6 mm
- added copper zone on F.Cu, net С6
Changed lines of the file:
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@@
   (general
     (links 149)
-    (no_connects 122)
+    (no_connects 113)
     (area 41.956667 64.005 204.271429 157.640001)
     (thickness 1.6)
     (drawings 2)
-    (tracks 49)
+    (tracks 65)
     (zones 0)
     (modules 89)
@@
   )
   (module Pin_Headers:Pin_Header_Straight_1x01_Pitch2.54mm (layer F.Cu)
-    (at 144.78 112.8268)
+    (at 148.082 121.285)
     (descr "Through hole straight pin header, 1x01, 2.54mm pitch, single row")
     (tags "Through hole pin header THT 1x01 2.54mm single row")
@@
   )
   (module TO_SOT_Packages_SMD:SOT-23_Handsoldering (layer F.Cu)
-    (at 148.6662 111.3028 90)
+    (at 149.3012 109.7788 90)
     (descr "SOT-23, Handsoldering")
     (tags SOT-23)
@@
   )
   (module TO_SOT_Packages_SMD:SOT-23_Handsoldering (layer F.Cu)
-    (at 149.5044 117.7798 270)
+    (at 150.1394 116.2558 270)
     (descr "SOT-23, Handsoldering")
     (tags SOT-23)
@@
   )
   (module Pin_Headers:Pin_Header_Straight_1x01_Pitch2.54mm (layer F.Cu)
-    (at 150.3934 106.807)
+    (at 149.479 104.775)
     (descr "Through hole straight pin header, 1x01, 2.54mm pitch, single row")
     (tags "Through hole pin header THT 1x01 2.54mm single row")
@@
   )
   (module Pin_Headers:Pin_Header_Straight_1x01_Pitch2.54mm (layer F.Cu)
-    (at 137.414 106.5022)
+    (at 141.224 104.521)
     (descr "Through hole straight pin header, 1x01, 2.54mm pitch, single row")
     (tags "Through hole pin header THT 1x01 2.54mm single row")
@@
   (segment (start 72.505 117.25) (end 72.505 119.455) (width 0.33) (layer F.Cu) (net 1))
   (segment (start 72.505 119.455) (end 72.275 119.685) (width 0.33) (layer F.Cu) (net 1))
+  (segment (start 146.515 115.4938) (end 146.515 117.559) (width 0.33) (layer F.Cu) (net 2))
+  (segment (start 148.082 119.126) (end 148.082 121.285) (width 0.33) (layer F.Cu) (net 2))
+  (segment (start 146.515 117.559) (end 148.082 119.126) (width 0.33) (layer F.Cu) (net 2))
+  (segment (start 144.907 118.2268) (end 146.8222 118.2268) (width 0.33) (layer F.Cu) (net 2))
+  (segment (start 148.082 119.4866) (end 148.082 121.285) (width 0.33) (layer F.Cu) (net 2))
+  (segment (start 146.8222 118.2268) (end 148.082 119.4866) (width 0.33) (layer F.Cu) (net 2))
   (segment (start 122.174 116.3066) (end 123.909 116.3066) (width 0.33) (layer F.Cu) (net 2))
   (segment (start 123.909 116.3066) (end 124.714 117.1116) (width 0.33) (layer F.Cu) (net 2))
@@
   (segment (start 126.619 115.3566) (end 123.759 112.4966) (width 0.33) (layer F.Cu) (net 9))
   (segment (start 123.759 112.4966) (end 122.404 112.4966) (width 0.33) (layer F.Cu) (net 9))
+  (segment (start 149.3012 108.2788) (end 149.3012 104.9528) (width 0.33) (layer F.Cu) (net 23))
+  (segment (start 149.3012 104.9528) (end 149.479 104.775) (width 0.33) (layer F.Cu) (net 23))
   (segment (start 100.7872 121.6406) (end 100.7872 120.4976) (width 0.33) (layer F.Cu) (net 23))
   (segment (start 101.3982 119.8866) (end 101.3982 118.0084) (width 0.33) (layer F.Cu) (net 23))
@@
   (segment (start 75.6502 106.435) (end 76.2254 107.0102) (width 0.33) (layer F.Cu) (net 23))
   (segment (start 110.109 112.4966) (end 113.054 112.4966) (width 0.33) (layer F.Cu) (net 23))
+  (segment (start 141.1986 107.7454) (end 141.1986 104.5464) (width 0.33) (layer F.Cu) (net 24))
+  (segment (start 141.1986 104.5464) (end 141.224 104.521) (width 0.33) (layer F.Cu) (net 24))
   (segment (start 100.711 109.474) (end 100.711 112.6222) (width 0.33) (layer F.Cu) (net 24))
   (segment (start 100.711 112.6222) (end 101.3728 113.284) (width 0.33) (layer F.Cu) (net 24))
@@
   (segment (start 96.4946 112.0394) (end 96.4946 113.3856) (width 0.33) (layer F.Cu) (net 38))
   (segment (start 95.697 111.2418) (end 96.4946 112.0394) (width 0.33) (layer F.Cu) (net 38))
+  (segment (start 149.1894 114.7558) (end 149.1894 114.0816) (width 0.33) (layer F.Cu) (net 42))
+  (segment (start 149.1894 114.0816) (end 150.2512 113.0198) (width 0.33) (layer F.Cu) (net 42))
+  (segment (start 150.2512 113.0198) (end 150.2512 111.2788) (width 0.33) (layer F.Cu) (net 42))
   (segment (start 116.054 111.5466) (end 116.779 111.5466) (width 0.33) (layer F.Cu) (net 47))
   (segment (start 116.779 111.5466) (end 118.679 113.4466) (width 0.33) (layer F.Cu) (net 47))
@@
   (segment (start 123.909 120.1166) (end 126.769 117.2566) (width 0.33) (layer F.Cu) (net 48))
   (segment (start 126.769 117.2566) (end 127.024 117.2566) (width 0.33) (layer F.Cu) (net 48))
+  (segment (start 139.8168 114.3748) (end 139.8168 113.8022) (width 0.33) (layer F.Cu) (net 49))
+  (segment (start 139.8168 113.8022) (end 142.1486 111.4704) (width 0.33) (layer F.Cu) (net 49))
+  (segment (start 142.1486 111.4704) (end 142.1486 110.7454) (width 0.33) (layer F.Cu) (net 49))
   (segment (start 116.054 119.1666) (end 116.779 119.1666) (width 0.33) (layer F.Cu) (net 51))
   (segment (start 116.779 119.1666) (end 118.679 121.0666) (width 0.33) (layer F.Cu) (net 51))
@@
       )
     )
+  )
+  (zone (net 21) (net_name С6) (layer F.Cu) (hatch edge 0.508)
+    (connect_pads (clearance 0.508))
+    (min_thickness 0.254)
+    (fill yes (arc_segments 16) (thermal_gap 0.508) (thermal_bridge_width 0.508))
+    (polygon
+      (pts
+        (xy 136.906 107.696) (xy 136.906 100.457) (xy 154.051 100.584) (xy 154.051 116.078) (xy 136.906 115.697)
+        (xy 136.525 113.411)
+      )
+    )
