File: Circuit/Mala.kicad_pcb (KiCad board)
At the start: 2 copper layers, 89 parts, among them J1 CONN_01X01, J10 CONN_01X01, J11 CONN_01X01, J12 CONN_01X01, J13 CONN_01X01, J14 CONN_01X01, J15 CONN_01X01, J16 CONN_01X01, J17 CONN_01X01, J18 CONN_01X01, J19 CONN_01X01, J2 CONN_01X01, J20 CONN_01X01, J21 CONN_01X01, J22 CONN_01X01, J23 CONN_01X01, J24 CONN_01X01, J25 CONN_01X01, J26 CONN_01X01, J27 CONN_01X01, J28 CONN_01X01, J29 CONN_01X01, J3 CONN_01X01, J30 CONN_01X01, J31 CONN_01X01, J32 CONN_01X01, J33 CONN_01X01, J4 CONN_01X01, J5 CONN_01X01, J6 CONN_02X08, J7 CONN_01X01, J8 CONN_01X01, J9 CONN_01X01, Q1 Q_NMOS_GSD, Q10 Q_NMOS_GSD, Q11 Q_NMOS_GSD, Q12 Q_NMOS_GSD, Q13 Q_NMOS_GSD, Q14 Q_NMOS_GSD, Q15 Q_NMOS_GSD, Q16 Q_NMOS_GSD, Q17 Q_NMOS_GSD, Q18 Q_NMOS_GSD, Q19 Q_NMOS_GSD, Q2 Q_NMOS_GSD, Q20 Q_NMOS_GSD, Q21 Q_NMOS_GSD, Q22 Q_NMOS_GSD, Q23 Q_NMOS_GSD, Q24 Q_NMOS_GSD, Q25 Q_NMOS_GSD, Q26 Q_NMOS_GSD, Q27 Q_NMOS_GSD, Q28 Q_NMOS_GSD, Q29 Q_NMOS_GSD, Q3 Q_NMOS_GSD, Q30 Q_NMOS_GSD, Q31 Q_NMOS_GSD, Q32 Q_NMOS_GSD, Q33 Q_NMOS_GSD, Q34 Q_NMOS_GSD, Q35 Q_NMOS_GSD, Q36 Q_NMOS_GSD, Q37 Q_NMOS_GSD, Q38 Q_NMOS_GSD, Q39 Q_NMOS_GSD, Q4 Q_NMOS_GSD, Q40 Q_NMOS_GSD, Q5 Q_NMOS_GSD, Q6 Q_NMOS_GSD, Q7 Q_NMOS_GSD, Q8 Q_NMOS_GSD, Q9 Q_NMOS_GSD

Commit message: 3 zones left
Parts:
- moved J26 49.7 mm to (65.8, 95.5)
- moved J25 38.8 mm to (80.0, 95.5)
Routing:
- net Net-(Q16-Pad3): track 0.00 -> 19.0 mm
- net Net-(C2-Pad1): track 0.00 -> 6.90 mm
- net Net-(J1-Pad1): track 0.00 -> 4.77 mm
- net Net-(Q15-Pad2): track 0.00 -> 4.14 mm
- net Net-(Q4-Pad2): track 0.00 -> 4.14 mm
- net Vcntrl: track 14.4 -> 18.4 mm
- net Vfb: track 14.6 -> 18.4 mm
- added copper zone on F.Cu, net GND
- added copper zone on F.Cu, net С1
Changed lines of the file:
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@@
   (general
     (links 149)
-    (no_connects 113)
-    (area 41.956667 64.005 204.271429 157.640001)
+    (no_connects 99)
+    (area 41.956667 75.9 204.271429 157.640001)
     (thickness 1.6)
     (drawings 2)
-    (tracks 65)
+    (tracks 91)
     (zones 0)
     (modules 89)
@@
   )
   (module Pin_Headers:Pin_Header_Straight_1x01_Pitch2.54mm (layer F.Cu)
-    (at 106.68 67.31)
+    (at 80.01 95.504)
     (descr "Through hole straight pin header, 1x01, 2.54mm pitch, single row")
     (tags "Through hole pin header THT 1x01 2.54mm single row")
@@
   )
   (module Pin_Headers:Pin_Header_Straight_1x01_Pitch2.54mm (layer F.Cu)
-    (at 106.68 67.31)
+    (at 65.786 95.504)
     (descr "Through hole straight pin header, 1x01, 2.54mm pitch, single row")
     (tags "Through hole pin header THT 1x01 2.54mm single row")
@@
   (segment (start 122.174 116.3066) (end 123.759 116.3066) (width 0.33) (layer F.Cu) (net 2))
   (segment (start 123.759 116.3066) (end 124.714 115.3516) (width 0.33) (layer F.Cu) (net 2))
+  (segment (start 69.85 86.13) (end 70.08 86.13) (width 0.33) (layer F.Cu) (net 3))
+  (segment (start 70.08 86.13) (end 71.44 84.77) (width 0.33) (layer F.Cu) (net 3))
+  (segment (start 71.44 84.77) (end 72.39 84.77) (width 0.33) (layer F.Cu) (net 3))
+  (segment (start 69.85 86.13) (end 69.85 84.328) (width 0.33) (layer F.Cu) (net 3))
+  (segment (start 69.3688 83.8468) (end 69.3688 82.5348) (width 0.33) (layer F.Cu) (net 3))
+  (segment (start 69.85 84.328) (end 69.3688 83.8468) (width 0.33) (layer F.Cu) (net 3))
   (segment (start 127.024 115.3566) (end 126.619 115.3566) (width 0.33) (layer F.Cu) (net 9))
   (segment (start 126.619 115.3566) (end 123.759 112.4966) (width 0.33) (layer F.Cu) (net 9))
   (segment (start 123.759 112.4966) (end 122.404 112.4966) (width 0.33) (layer F.Cu) (net 9))
+  (segment (start 64.9605 85.7758) (end 64.9605 82.9931) (width 0.33) (layer F.Cu) (net 10) (status 400000))
+  (segment (start 64.9605 82.9931) (end 66.3688 81.5848) (width 0.33) (layer F.Cu) (net 10) (status 800000))
+  (segment (start 65.786 95.504) (end 69.826 95.504) (width 0.33) (layer F.Cu) (net 23))
+  (segment (start 69.826 95.504) (end 69.85 95.48) (width 0.33) (layer F.Cu) (net 23))
   (segment (start 149.3012 108.2788) (end 149.3012 104.9528) (width 0.33) (layer F.Cu) (net 23))
   (segment (start 149.3012 104.9528) (end 149.479 104.775) (width 0.33) (layer F.Cu) (net 23))
@@
   (segment (start 75.6502 106.435) (end 76.2254 107.0102) (width 0.33) (layer F.Cu) (net 23))
   (segment (start 110.109 112.4966) (end 113.054 112.4966) (width 0.33) (layer F.Cu) (net 23))
+  (segment (start 76.2 95.48) (end 79.986 95.48) (width 0.33) (layer F.Cu) (net 24))
+  (segment (start 79.986 95.48) (end 80.01 95.504) (width 0.33) (layer F.Cu) (net 24))
   (segment (start 141.1986 107.7454) (end 141.1986 104.5464) (width 0.33) (layer F.Cu) (net 24))
   (segment (start 141.1986 104.5464) (end 141.224 104.521) (width 0.33) (layer F.Cu) (net 24))
@@
   (segment (start 73.455 110.045) (end 71.555 111.945) (width 0.33) (layer F.Cu) (net 28))
   (segment (start 71.555 111.945) (end 71.555 112.785) (width 0.33) (layer F.Cu) (net 28))
+  (segment (start 68.9 92.48) (end 68.9 92.136) (width 0.33) (layer F.Cu) (net 30))
+  (segment (start 68.9 92.136) (end 70.8 90.236) (width 0.33) (layer F.Cu) (net 30))
+  (segment (start 70.8 90.236) (end 70.8 89.13) (width 0.33) (layer F.Cu) (net 30))
+  (segment (start 72.39 78.91) (end 77.894 78.91) (width 0.33) (layer F.Cu) (net 31))
+  (segment (start 78.208 86.13) (end 76.2 86.13) (width 0.33) (layer F.Cu) (net 31))
+  (segment (start 78.74 85.598) (end 78.208 86.13) (width 0.33) (layer F.Cu) (net 31))
+  (segment (start 78.74 79.756) (end 78.74 85.598) (width 0.33) (layer F.Cu) (net 31))
+  (segment (start 77.894 78.91) (end 78.74 79.756) (width 0.33) (layer F.Cu) (net 31))
+  (segment (start 69.3688 80.6348) (end 70.2412 80.6348) (width 0.33) (layer F.Cu) (net 31))
+  (segment (start 70.2412 80.6348) (end 71.966 78.91) (width 0.33) (layer F.Cu) (net 31))
+  (segment (start 71.966 78.91) (end 72.39 78.91) (width 0.33) (layer F.Cu) (net 31))
   (segment (start 94.2354 118.938) (end 98.3778 118.938) (width 0.33) (layer F.Cu) (net 32))
   (segment (start 98.3778 118.938) (end 98.3982 118.9584) (width 0.33) (layer F.Cu) (net 32))
@@
   (segment (start 67.105 109.995) (end 65.205 111.895) (width 0.33) (layer F.Cu) (net 34))
   (segment (start 65.205 111.895) (end 65.205 112.785) (width 0.33) (layer F.Cu) (net 34))
+  (segment (start 75.25 92.48) (end 75.25 91.882) (width 0.33) (layer F.Cu) (net 37))
+  (segment (start 75.25 91.882) (end 77.15 89.982) (width 0.33) (layer F.Cu) (net 37))
+  (segment (start 77.15 89.982) (end 77.15 89.13) (width 0.33) (layer F.Cu) (net 37))
   (segment (start 94.6418 111.2418) (end 95.697 111.2418) (width 0.33) (layer F.Cu) (net 38))
   (segment (start 97.343 114.234) (end 98.3728 114.234) (width 0.33) (layer F.Cu) (net 38))
@@
       )
     )
+  )
+  (zone (net 2) (net_name GND) (layer F.Cu) (hatch edge 0.508)
+    (connect_pads (clearance 0.508))
+    (min_thickness 0.254)
+    (fill yes (arc_segments 16) (thermal_gap 0.508) (thermal_bridge_width 0.508))
+    (polygon
+      (pts
+        (xy 71.374 80.772) (xy 73.66 79.756) (xy 77.216 79.756) (xy 77.978 80.264) (xy 77.978 83.566)
+        (xy 77.216 84.074) (xy 74.168 84.074) (xy 73.406 83.312) (xy 71.628 83.312) (xy 71.374 82.804)
+      )
+    )
+  )
+  (zone (net 16) (net_name С1) (layer F.Cu) (hatch edge 0.508)
+    (connect_pads (clearance 0.508))
+    (min_thickness 0.254)
+    (fill yes (arc_segments 16) (thermal_gap 0.508) (thermal_bridge_width 0.508))
+    (polygon
+      (pts
+        (xy 62.23 93.726) (xy 67.818 88.138) (xy 78.994 88.138) (xy 82.804 93.726) (xy 82.804 97.028)
+        (xy 81.788 98.044) (xy 63.5 98.044) (xy 62.23 96.774) (xy 62.23 96.012)
+      )
+    )

Commit message: 2 zones left
Parts:
- moved J21 6.15 mm to (98.6, 79.0)
- moved Q21 4.64 mm to (129.0, 84.6)
- moved Q29 4.64 mm to (129.0, 92.8)
- moved C5 4.64 mm to (139.8, 86.5)
- moved J27 4.64 mm to (131.6, 88.4)
- moved Q22 4.64 mm to (135.4, 84.6)
- moved Q30 4.64 mm to (135.4, 92.8)
- moved R5 4.64 mm to (139.8, 90.3)
- moved Q20 3.45 mm to (91.2, 82.6)
- moved Q19 3.45 mm to (97.5, 82.6)
- moved R4 2.93 mm to (88.4, 85.9)
- moved J3 2.84 mm to (82.5, 78.7)
- moved Q12 2.75 mm to (97.4, 92.1)
- moved Q13 2.75 mm to (90.8, 92.0)
- moved J20 2.49 mm to (99.1, 88.4)
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Routing:
- net Net-(C4-Pad1): track 0.00 -> 8.48 mm
- net Net-(Q14-Pad2): track 0.00 -> 7.01 mm
- net GND: track 17.7 -> 23.0 mm
- net Net-(Q12-Pad2): track 0.00 -> 4.49 mm
- net Net-(Q19-Pad2): track 0.00 -> 4.18 mm
- added copper zone on F.Cu, net С3
Changed lines of the file:
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@@
   (general
     (links 149)
-    (no_connects 99)
+    (no_connects 88)
     (area 41.956667 75.9 204.271429 157.640001)
     (thickness 1.6)
     (drawings 2)
-    (tracks 91)
+    (tracks 115)
     (zones 0)
     (modules 89)
@@
   )
   (module Capacitors_SMD:C_0603_HandSoldering (layer F.Cu)
-    (at 135.255 85.725 270)
+    (at 139.827 86.487 270)
     (descr "Capacitor SMD 0603, hand soldering")
     (tags "capacitor 0603")
@@
   )
   (module Pin_Headers:Pin_Header_Straight_1x01_Pitch2.54mm (layer F.Cu)
-    (at 84.5566 80.7466)
+    (at 82.55 78.74)
     (descr "Through hole straight pin header, 1x01, 2.54mm pitch, single row")
     (tags "Through hole pin header THT 1x01 2.54mm single row")
@@
   )
   (module Pin_Headers:Pin_Header_Straight_1x01_Pitch2.54mm (layer F.Cu)
-    (at 93.8022 85.2805)
+    (at 93.218 87.376)
     (descr "Through hole straight pin header, 1x01, 2.54mm pitch, single row")
     (tags "Through hole pin header THT 1x01 2.54mm single row")
@@
   )
   (module TO_SOT_Packages_SMD:SOT-23_Handsoldering (layer F.Cu)
-    (at 95.12935 93.65615)
+    (at 97.41535 92.13215)
     (descr "SOT-23, Handsoldering")
     (tags SOT-23)
@@
   )
   (module TO_SOT_Packages_SMD:SOT-23_Handsoldering (layer F.Cu)
-    (at 88.48725 93.50375 180)
+    (at 90.77325 91.97975 180)
     (descr "SOT-23, Handsoldering")
     (tags SOT-23)
@@
   )
   (module TO_SOT_Packages_SMD:SOT-23_Handsoldering (layer F.Cu)
-    (at 86.0044 86.1695 180)
+    (at 84.328 87.63 180)
     (descr "SOT-23, Handsoldering")
     (tags SOT-23)
@@
   )
   (module TO_SOT_Packages_SMD:SOT-23_Handsoldering (layer F.Cu)
-    (at 99.57435 79.82585)
+    (at 97.54235 82.61985)
     (descr "SOT-23, Handsoldering")
     (tags SOT-23)
@@
   )
   (module TO_SOT_Packages_SMD:SOT-23_Handsoldering (layer F.Cu)
-    (at 93.19895 79.77505 180)
+    (at 91.16695 82.56905 180)
     (descr "SOT-23, Handsoldering")
     (tags SOT-23)
@@
   )
   (module TO_SOT_Packages_SMD:SOT-23_Handsoldering (layer F.Cu)
-    (at 124.46 83.82 180)
+    (at 129.032 84.582 180)
     (descr "SOT-23, Handsoldering")
     (tags SOT-23)
@@
   )
   (module TO_SOT_Packages_SMD:SOT-23_Handsoldering (layer F.Cu)
-    (at 130.81 83.82)
+    (at 135.382 84.582)
     (descr "SOT-23, Handsoldering")
     (tags SOT-23)
@@
   )
   (module TO_SOT_Packages_SMD:SOT-23_Handsoldering (layer F.Cu)
-    (at 124.46 92.075 180)
+    (at 129.032 92.837 180)
     (descr "SOT-23, Handsoldering")
     (tags SOT-23)
@@
   )
   (module TO_SOT_Packages_SMD:SOT-23_Handsoldering (layer F.Cu)
-    (at 130.81 92.075)
+    (at 135.382 92.837)
     (descr "SOT-23, Handsoldering")
     (tags SOT-23)
@@
   )
   (module Resistors_SMD:R_0603_HandSoldering (layer F.Cu)
-    (at 90.2335 83.5787 270)
+    (at 88.392 85.852 270)
     (descr "Resistor SMD 0603, hand soldering")
     (tags "resistor 0603")
@@
   )
   (module Resistors_SMD:R_0603_HandSoldering (layer F.Cu)
-    (at 135.255 89.535 90)
+    (at 139.827 90.297 90)
     (descr "Resistor SMD 0603, hand soldering")
     (tags "resistor 0603")
@@
   )
   (module Pin_Headers:Pin_Header_Straight_1x01_Pitch2.54mm (layer F.Cu)
-    (at 96.901 89.6239)
+    (at 99.06 88.392)
     (descr "Through hole straight pin header, 1x01, 2.54mm pitch, single row")
     (tags "Through hole pin header THT 1x01 2.54mm single row")
@@
   )
   (module Pin_Headers:Pin_Header_Straight_1x01_Pitch2.54mm (layer F.Cu)
-    (at 97.6503 85.0773)
+    (at 98.552 78.994)
     (descr "Through hole straight pin header, 1x01, 2.54mm pitch, single row")
     (tags "Through hole pin header THT 1x01 2.54mm single row")
@@
   )
   (module Pin_Headers:Pin_Header_Straight_1x01_Pitch2.54mm (layer F.Cu)
-    (at 127 87.63)
+    (at 131.572 88.392)
     (descr "Through hole straight pin header, 1x01, 2.54mm pitch, single row")
     (tags "Through hole pin header THT 1x01 2.54mm single row")
@@
   (segment (start 72.505 117.25) (end 72.505 119.455) (width 0.33) (layer F.Cu) (net 1))
   (segment (start 72.505 119.455) (end 72.275 119.685) (width 0.33) (layer F.Cu) (net 1))
+  (segment (start 88.392 86.952) (end 89.324 86.952) (width 0.33) (layer F.Cu) (net 2))
+  (segment (start 89.5833 86.6927) (end 90.2335 86.6927) (width 0.33) (layer F.Cu) (net 2))
+  (segment (start 89.324 86.952) (end 89.5833 86.6927) (width 0.33) (layer F.Cu) (net 2))
+  (segment (start 93.218 87.376) (end 92.456 87.376) (width 0.33) (layer F.Cu) (net 2))
+  (segment (start 92.456 87.376) (end 91.7727 86.6927) (width 0.33) (layer F.Cu) (net 2))
+  (segment (start 91.7727 86.6927) (end 90.2335 86.6927) (width 0.33) (layer F.Cu) (net 2))
   (segment (start 146.515 115.4938) (end 146.515 117.559) (width 0.33) (layer F.Cu) (net 2))
   (segment (start 148.082 119.126) (end 148.082 121.285) (width 0.33) (layer F.Cu) (net 2))
@@
   (segment (start 69.3688 83.8468) (end 69.3688 82.5348) (width 0.33) (layer F.Cu) (net 3))
   (segment (start 69.85 84.328) (end 69.3688 83.8468) (width 0.33) (layer F.Cu) (net 3))
+  (segment (start 89.27325 91.97975) (end 88.93175 91.97975) (width 0.33) (layer F.Cu) (net 5))
+  (segment (start 88.93175 91.97975) (end 88.138 91.186) (width 0.33) (layer F.Cu) (net 5))
+  (segment (start 88.138 91.186) (end 88.138 88.58) (width 0.33) (layer F.Cu) (net 5))
+  (segment (start 85.828 88.58) (end 88.138 88.58) (width 0.33) (layer F.Cu) (net 5))
+  (segment (start 88.138 88.58) (end 90.2208 88.58) (width 0.33) (layer F.Cu) (net 5))
+  (segment (start 90.2208 88.58) (end 90.2335 88.5927) (width 0.33) (layer F.Cu) (net 5))
   (segment (start 127.024 115.3566) (end 126.619 115.3566) (width 0.33) (layer F.Cu) (net 9))
   (segment (start 126.619 115.3566) (end 123.759 112.4966) (width 0.33) (layer F.Cu) (net 9))
   (segment (start 123.759 112.4966) (end 122.404 112.4966) (width 0.33) (layer F.Cu) (net 9))
-  (segment (start 64.9605 85.7758) (end 64.9605 82.9931) (width 0.33) (layer F.Cu) (net 10) (status 400000))
-  (segment (start 64.9605 82.9931) (end 66.3688 81.5848) (width 0.33) (layer F.Cu) (net 10) (status 800000))
+  (segment (start 64.9605 85.7758) (end 64.9605 82.9931) (width 0.33) (layer F.Cu) (net 10))
+  (segment (start 64.9605 82.9931) (end 66.3688 81.5848) (width 0.33) (layer F.Cu) (net 10))
   (segment (start 65.786 95.504) (end 69.826 95.504) (width 0.33) (layer F.Cu) (net 23))
   (segment (start 69.826 95.504) (end 69.85 95.48) (width 0.33) (layer F.Cu) (net 23))
@@
   (segment (start 67.105 109.995) (end 65.205 111.895) (width 0.33) (layer F.Cu) (net 34))
   (segment (start 65.205 111.895) (end 65.205 112.785) (width 0.33) (layer F.Cu) (net 34))
+  (segment (start 92.27325 91.02975) (end 93.06175 91.02975) (width 0.33) (layer F.Cu) (net 35))
+  (segment (start 93.06175 91.02975) (end 95.11415 93.08215) (width 0.33) (layer F.Cu) (net 35))
+  (segment (start 95.11415 93.08215) (end 95.91535 93.08215) (width 0.33) (layer F.Cu) (net 35))
+  (segment (start 85.828 86.68) (end 85.828 85.876) (width 0.33) (layer F.Cu) (net 36))
+  (segment (start 86.952 84.752) (end 88.392 84.752) (width 0.33) (layer F.Cu) (net 36))
+  (segment (start 85.828 85.876) (end 86.952 84.752) (width 0.33) (layer F.Cu) (net 36))
+  (segment (start 88.392 84.752) (end 88.392 83.058) (width 0.33) (layer F.Cu) (net 36))
+  (segment (start 88.392 83.058) (end 88.88095 82.56905) (width 0.33) (layer F.Cu) (net 36))
+  (segment (start 88.88095 82.56905) (end 89.66695 82.56905) (width 0.33) (layer F.Cu) (net 36))
   (segment (start 75.25 92.48) (end 75.25 91.882) (width 0.33) (layer F.Cu) (net 37))
   (segment (start 75.25 91.882) (end 77.15 89.982) (width 0.33) (layer F.Cu) (net 37))
@@
   (segment (start 96.4946 112.0394) (end 96.4946 113.3856) (width 0.33) (layer F.Cu) (net 38))
   (segment (start 95.697 111.2418) (end 96.4946 112.0394) (width 0.33) (layer F.Cu) (net 38))
+  (segment (start 92.66695 81.61905) (end 93.30305 81.61905) (width 0.33) (layer F.Cu) (net 39))
+  (segment (start 93.30305 81.61905) (end 95.25385 83.56985) (width 0.33) (layer F.Cu) (net 39))
+  (segment (start 95.25385 83.56985) (end 96.04235 83.56985) (width 0.33) (layer F.Cu) (net 39))
   (segment (start 149.1894 114.7558) (end 149.1894 114.0816) (width 0.33) (layer F.Cu) (net 42))
   (segment (start 149.1894 114.0816) (end 150.2512 113.0198) (width 0.33) (layer F.Cu) (net 42))
@@
       )
     )
+  )
+  (zone (net 18) (net_name С3) (layer F.Cu) (hatch edge 0.508)
+    (connect_pads (clearance 0.508))
+    (min_thickness 0.254)
+    (fill yes (arc_segments 16) (thermal_gap 0.508) (thermal_bridge_width 0.508))
+    (polygon
+      (pts
+        (xy 90.17 84.836) (xy 90.17 76.454) (xy 101.346 76.454) (xy 101.346 94.488) (xy 90.17 94.742)
+        (xy 90.17 92.964)
+      )
+    )
