File: Circuit/Mala.kicad_pcb (KiCad board)
At the start: 2 copper layers, 89 parts, among them J1 CONN_01X01, J10 CONN_01X01, J11 CONN_01X01, J12 CONN_01X01, J13 CONN_01X01, J14 CONN_01X01, J15 CONN_01X01, J16 CONN_01X01, J17 CONN_01X01, J18 CONN_01X01, J19 CONN_01X01, J2 CONN_01X01, J20 CONN_01X01, J21 CONN_01X01, J22 CONN_01X01, J23 CONN_01X01, J24 CONN_01X01, J25 CONN_01X01, J26 CONN_01X01, J27 CONN_01X01, J28 CONN_01X01, J29 CONN_01X01, J3 CONN_01X01, J30 CONN_01X01, J31 CONN_01X01, J32 CONN_01X01, J33 CONN_01X01, J4 CONN_01X01, J5 CONN_01X01, J6 CONN_02X08, J7 CONN_01X01, J8 CONN_01X01, J9 CONN_01X01, Q1 Q_NMOS_GSD, Q10 Q_NMOS_GSD, Q11 Q_NMOS_GSD, Q12 Q_NMOS_GSD, Q13 Q_NMOS_GSD, Q14 Q_NMOS_GSD, Q15 Q_NMOS_GSD, Q16 Q_NMOS_GSD, Q17 Q_NMOS_GSD, Q18 Q_NMOS_GSD, Q19 Q_NMOS_GSD, Q2 Q_NMOS_GSD, Q20 Q_NMOS_GSD, Q21 Q_NMOS_GSD, Q22 Q_NMOS_GSD, Q23 Q_NMOS_GSD, Q24 Q_NMOS_GSD, Q25 Q_NMOS_GSD, Q26 Q_NMOS_GSD, Q27 Q_NMOS_GSD, Q28 Q_NMOS_GSD, Q29 Q_NMOS_GSD, Q3 Q_NMOS_GSD, Q30 Q_NMOS_GSD, Q31 Q_NMOS_GSD, Q32 Q_NMOS_GSD, Q33 Q_NMOS_GSD, Q34 Q_NMOS_GSD, Q35 Q_NMOS_GSD, Q36 Q_NMOS_GSD, Q37 Q_NMOS_GSD, Q38 Q_NMOS_GSD, Q39 Q_NMOS_GSD, Q4 Q_NMOS_GSD, Q40 Q_NMOS_GSD, Q5 Q_NMOS_GSD, Q6 Q_NMOS_GSD, Q7 Q_NMOS_GSD, Q8 Q_NMOS_GSD, Q9 Q_NMOS_GSD

Commit message: 1 zone left
Parts:
- moved J11 94.2 mm to (139.2, 87.4)
- moved J33 9.86 mm to (119.6, 91.4)
- moved J28 6.37 mm to (129.5, 87.1)
- moved J27 5.71 mm to (128.5, 93.2)
- moved Q27 5.71 mm to (110.7, 90.7)
- moved Q29 5.40 mm to (133.9, 90.4)
- moved Q30 5.10 mm to (140.2, 91.2)
- moved J8 4.93 mm to (150.2, 84.1)
- moved Q21 4.93 mm to (133.9, 83.6)
- moved Q22 4.93 mm to (140.2, 83.6)
- moved Q23 4.93 mm to (151.5, 90.4)
- moved C5 4.19 mm to (144.0, 86.4)
- moved Q28 4.02 mm to (108.7, 84.1)
- moved C7 3.88 mm to (111.3, 80.5)
- moved J32 3.71 mm to (106.9, 91.7)
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Routing:
- net Net-(C7-Pad1): track 0.00 -> 8.92 mm
- net Net-(Q31-Pad2): track 0.00 -> 5.77 mm
- net GND: track 23.0 -> 28.3 mm
- net Net-(Q37-Pad2): track 0.00 -> 4.60 mm
- net Vfb: track 18.4 -> 22.5 mm
- net Vcntrl: track 18.4 -> 22.5 mm
- net Net-(J7-Pad1): track 0.00 -> 3.69 mm
- net Net-(Q27-Pad2): track 0.00 -> 3.66 mm
- added copper zone on F.Cu, net С5
